File: led_status_pcb_design.kicad_pcb (KiCad board)
At the start: 2 copper layers, 65 x 30 mm, 5 parts, among them J1 GPIO_CONNECTOR

Commit message: Status LEDs PCB
Parts:
- added BT1: 5V supply, Battery:Battery_Panasonic_CR1025-VSK_Vertical_CircularHoles, F.Cu at (122.3, 104.7)
- added D1: CQY99, LED_THT:LED_D5.0mm_Horizontal_O1.27mm_Z3.0mm_IRGrey, B.Cu at (122.1, 109.8)
- added D10: CQY99, LED_THT:LED_D5.0mm_Horizontal_O1.27mm_Z3.0mm_IRGrey, B.Cu at (166.8, 109.8)
- added D2: CQY99, LED_THT:LED_D5.0mm_Horizontal_O1.27mm_Z3.0mm_IRGrey, B.Cu at (126.1, 109.8)
- added D3: CQY99, LED_THT:LED_D5.0mm_Horizontal_O1.27mm_Z3.0mm_IRGrey, F.Cu at (131.2, 109.8)
- added D4: CQY99, LED_THT:LED_D5.0mm_Horizontal_O1.27mm_Z3.0mm_IRGrey, B.Cu at (136.3, 109.8)
- added D5: CQY99, LED_THT:LED_D5.0mm_Horizontal_O1.27mm_Z3.0mm_IRGrey, F.Cu at (141.4, 109.8)
- added D6: CQY99, LED_THT:LED_D5.0mm_Horizontal_O1.27mm_Z3.0mm_IRGrey, B.Cu at (146.4, 109.8)
- added D7: CQY99, LED_THT:LED_D5.0mm_Horizontal_O1.27mm_Z3.0mm_IRGrey, F.Cu at (151.5, 109.8)
- added D8: CQY99, LED_THT:LED_D5.0mm_Horizontal_O1.27mm_Z3.0mm_IRGrey, B.Cu at (156.6, 109.8)
- added D9: CQY99, LED_THT:LED_D5.0mm_Horizontal_O1.27mm_Z3.0mm_IRGrey, F.Cu at (161.7, 109.8)
- added Q1: 2N2219, digikey-footprints:TO-39-3, F.Cu at (171.3, 115.9)
- added Q2: 2N3905, digikey-footprints:TO-92-3, B.Cu at (174.4, 111.1)
- added R1: 300, Resistor_THT:R_Axial_DIN0207_L6.3mm_D2.5mm_P7.62mm_Horizontal, F.Cu at (126.5, 99.1)
- added R10: 300, Resistor_THT:R_Axial_DIN0207_L6.3mm_D2.5mm_P7.62mm_Horizontal, F.Cu at (159.9, 99.0)
- added R11: 55, Resistor_THT:R_Axial_DIN0207_L6.3mm_D2.5mm_P7.62mm_Horizontal, F.Cu at (164.0, 98.6)
- added R12: 10, Resistor_THT:R_Axial_DIN0207_L6.3mm_D2.5mm_P7.62mm_Horizontal, F.Cu at (168.1, 98.6)
- added R13: 1k, Resistor_THT:R_Axial_DIN0207_L6.3mm_D2.5mm_P7.62mm_Horizontal, F.Cu at (171.9, 98.6)
- added R14: 22k, Resistor_THT:R_Axial_DIN0207_L6.3mm_D2.5mm_P7.62mm_Horizontal, F.Cu at (175.5, 98.6)
- added R15: 10k, Resistor_THT:R_Axial_DIN0207_L6.3mm_D2.5mm_P7.62mm_Horizontal, F.Cu at (179.2, 99.1)
- added R2: 300, Resistor_THT:R_Axial_DIN0207_L6.3mm_D2.5mm_P7.62mm_Horizontal, F.Cu at (130.1, 99.2)
- added R3: 300, Resistor_THT:R_Axial_DIN0207_L6.3mm_D2.5mm_P7.62mm_Horizontal, F.Cu at (133.7, 99.1)
- added R4: 300, Resistor_THT:R_Axial_DIN0207_L6.3mm_D2.5mm_P7.62mm_Horizontal, F.Cu at (137.3, 98.5)
- added R5: 300, Resistor_THT:R_Axial_DIN0207_L6.3mm_D2.5mm_P7.62mm_Horizontal, F.Cu at (141.3, 98.5)
- added R6: 300, Resistor_THT:R_Axial_DIN0207_L6.3mm_D2.5mm_P7.62mm_Horizontal, F.Cu at (145.0, 98.5)
- added R7: 300, Resistor_THT:R_Axial_DIN0207_L6.3mm_D2.5mm_P7.62mm_Horizontal, F.Cu at (148.3, 99.1)
- added R8: 300, Resistor_THT:R_Axial_DIN0207_L6.3mm_D2.5mm_P7.62mm_Horizontal, F.Cu at (152.1, 98.9)
- added R9: 300, Resistor_THT:R_Axial_DIN0207_L6.3mm_D2.5mm_P7.62mm_Horizontal, F.Cu at (156.1, 99.0)
- J1: moved to F.Cu
- moved J1 2.73 mm to (126.0, 93.1), turned to 90 degrees
Routing:
- net GND: track 0.00 -> 257.5 mm
- net +5V: track 0.00 -> 130.4 mm
- net +3V3: track 0.00 -> 60.1 mm
- net /GPIO17_GEN0: track 0.00 -> 30.1 mm
- net /GPIO26: track 0.00 -> 29.5 mm
- net /GPIO5: track 0.00 -> 28.6 mm
- net /GPIO6: track 0.00 -> 25.6 mm
- net Net-(Q2-Pad3): track 0.00 -> 24.5 mm
- net Net-(Q1-Pad2): track 0.00 -> 15.7 mm
- net /GPIO27_GEN2: track 0.00 -> 14.0 mm
- net /GPIO22_GEN3: track 0.00 -> 12.9 mm
- net Net-(Q1-Pad3): track 0.00 -> 11.9 mm
- net /GPIO16: track 0.00 -> 11.3 mm
- net Net-(D10-Pad2): track 0.00 -> 10.9 mm
- net Net-(D1-Pad2): track 0.00 -> 10.9 mm
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Other:
- board text removed: "Board dimensions are on Cmts (Comments) layer. Deselect it in Layers Manager to make them invisible. GPIO connector nets are not connected, these will get updated as per your schematic/netlist."
